File: source/Power.sch (KiCad schematic (older format))
At the start: 60 parts, among them J4 On/Off, U1 AMS1117-3.3, U2 DRV8301, U3 TP2604-SR

Commit message: started redrawing pcb
Parts:
- C10, C11, C20, C21, C22, C9: footprint Capacitor_SMD:C_0805_2012Metric -> Capacitor_SMD:C_0603_1608Metric
- C12, C13, C14, C16, C17, C18, C19, C23, C24, C25, C26, C27, C28, C29, C30, C32, C33, C34, C57, C58, C59, C7, C8: footprint Capacitor_SMD:C_0603_1608Metric -> Capacitor_SMD:C_0402_1005Metric
- C15, C31: footprint Capacitor_SMD:C_1210_3225Metric -> Capacitor_SMD:C_1210_3225Metric_Pad1.42x2.65mm_HandSolder
- R18, R19, R20, R21, R22, R23, R24, R25, R26, R27, R28, R29, R30, R31, R32, R36, R38, R64, R65, R66, R67: footprint Resistor_SMD:R_0603_1608Metric -> Resistor_SMD:R_0402_1005Metric
