File: source/hall_filters.sch (KiCad schematic (older format))
At the start: 5 parts

Commit message: started redrawing pcb
Parts:
- C6: footprint Capacitor_SMD:C_0603_1608Metric -> Capacitor_SMD:C_0402_1005Metric
- R14, R15, R16, R17: footprint Resistor_SMD:R_0603_1608Metric -> Resistor_SMD:R_0402_1005Metric
Changed lines of the file:
@@
 $Descr User 8496 6906
 encoding utf-8
-Sheet 3 8
+Sheet 3 6
 Title "Cheap FOCer 2"
 Date "2020-04-08"
@@
 F 0 "R14" V 3700 2700 50  0000 C CNN
 F 1 "10k" V 3600 2700 50  0000 C CNN
-F 2 "Resistor_SMD:R_0603_1608Metric" H 3600 2700 60  0001 C CNN
+F 2 "Resistor_SMD:R_0402_1005Metric" H 3600 2700 60  0001 C CNN
 F 3 "" H 3600 2700 60  0001 C CNN
 	1    3600 2700
@@
 F 0 "R15" V 3900 2700 50  0000 C CNN
 F 1 "2k2" V 3800 2700 50  0000 C CNN
-F 2 "Resistor_SMD:R_0603_1608Metric" H 3800 2700 60  0001 C CNN
+F 2 "Resistor_SMD:R_0402_1005Metric" H 3800 2700 60  0001 C CNN
 F 3 "" H 3800 2700 60  0001 C CNN
 	1    3800 2700
@@
 F 0 "R16" V 4100 2700 50  0000 C CNN
 F 1 "2k2" V 4000 2700 50  0000 C CNN
-F 2 "Resistor_SMD:R_0603_1608Metric" H 4000 2700 60  0001 C CNN
+F 2 "Resistor_SMD:R_0402_1005Metric" H 4000 2700 60  0001 C CNN
 F 3 "" H 4000 2700 60  0001 C CNN
 	1    4000 2700
@@
 F 0 "R17" V 4300 2700 50  0000 C CNN
 F 1 "2k2" V 4200 2700 50  0000 C CNN
-F 2 "Resistor_SMD:R_0603_1608Metric" H 4200 2700 60  0001 C CNN
+F 2 "Resistor_SMD:R_0402_1005Metric" H 4200 2700 60  0001 C CNN
 F 3 "" H 4200 2700 60  0001 C CNN
 	1    4200 2700
@@
 F 0 "C6" H 4000 3550 50  0000 L CNN
 F 1 "100n" H 3950 3650 50  0000 L CNN
-F 2 "Capacitor_SMD:C_0603_1608Metric" H 4250 3550 60  0001 C CNN
+F 2 "Capacitor_SMD:C_0402_1005Metric" H 4250 3550 60  0001 C CNN
 F 3 "" H 4250 3550 60  0001 C CNN
 	1    4250 3550
