File: source/mosfets.sch (KiCad schematic (older format))
At the start: 50 parts, among them Q1 NCEP60T20, Q2 NCEP60T20, Q3 NCEP60T20, Q4 NCEP60T20, Q5 NCEP60T20, Q6 NCEP60T20

Commit message: started redrawing pcb
Parts:
- C40, C41, C42: footprint Capacitor_SMD:C_0805_2012Metric -> Capacitor_SMD:C_0805_2012Metric_Pad1.15x1.40mm_HandSolder
- C61, C62, C63, C65, C66, C67: footprint Capacitor_SMD:C_0603_1608Metric -> Capacitor_SMD:C_0402_1005Metric
- R37: footprint Resistor_SMD:R_0805_2012Metric -> Resistor_SMD:R_0402_1005Metric
- R44, R45, R46, R50, R51, R52: footprint Resistor_SMD:R_0603_1608Metric -> Resistor_SMD:R_0402_1005Metric
Changed lines of the file:
@@
 $Descr A4 11693 8268
 encoding utf-8
-Sheet 5 8
+Sheet 5 6
 Title "Cheap FOCer 2"
 Date "2020-04-08"
@@
 F 0 "C40" H 4300 4250 50  0000 L CNN
 F 1 "4.7nF, 100V" H 4200 4050 50  0000 L CNN
-F 2 "Capacitor_SMD:C_0805_2012Metric" H 4450 4150 60  0001 C CNN
+F 2 "Capacitor_SMD:C_0805_2012Metric_Pad1.15x1.40mm_HandSolder" H 4450 4150 60  0001 C CNN
 F 3 "" H 4450 4150 60  0001 C CNN
 	1    4450 4150
@@
 F 0 "C41" H 6900 4300 50  0000 L CNN
 F 1 "4.7nF, 100V" H 6800 4100 50  0000 L CNN
-F 2 "Capacitor_SMD:C_0805_2012Metric" H 7050 4200 60  0001 C CNN
+F 2 "Capacitor_SMD:C_0805_2012Metric_Pad1.15x1.40mm_HandSolder" H 7050 4200 60  0001 C CNN
 F 3 "" H 7050 4200 60  0001 C CNN
 	1    7050 4200
@@
 F 0 "C42" H 9700 4350 50  0000 L CNN
 F 1 "4.7nF, 100V" H 9700 4150 50  0000 L CNN
-F 2 "Capacitor_SMD:C_0805_2012Metric" H 9650 4250 60  0001 C CNN
+F 2 "Capacitor_SMD:C_0805_2012Metric_Pad1.15x1.40mm_HandSolder" H 9650 4250 60  0001 C CNN
 F 3 "" H 9650 4250 60  0001 C CNN
 	1    9650 4250
@@
 F 0 "R50" V 3600 4700 50  0000 C CNN
 F 1 "4.7k" V 3500 4700 50  0000 C CNN
-F 2 "Resistor_SMD:R_0603_1608Metric" H 3500 4700 60  0001 C CNN
+F 2 "Resistor_SMD:R_0402_1005Metric" H 3500 4700 60  0001 C CNN
 F 3 "" H 3500 4700 60  0001 C CNN
 	1    3500 4700
@@
 F 0 "R52" V 8600 4750 50  0000 C CNN
 F 1 "4.7k" V 8700 4750 50  0000 C CNN
-F 2 "Resistor_SMD:R_0603_1608Metric" H 8700 4750 60  0001 C CNN
+F 2 "Resistor_SMD:R_0402_1005Metric" H 8700 4750 60  0001 C CNN
 F 3 "" H 8700 4750 60  0001 C CNN
 	1    8700 4750
@@
 F 0 "R44" V 3400 3650 50  0000 C CNN
 F 1 "4.7k" V 3500 3650 50  0000 C CNN
-F 2 "Resistor_SMD:R_0603_1608Metric" H 3500 3650 60  0001 C CNN
+F 2 "Resistor_SMD:R_0402_1005Metric" H 3500 3650 60  0001 C CNN
 F 3 "" H 3500 3650 60  0001 C CNN
 	1    3500 3650
@@
 F 0 "R46" V 8800 3750 50  0000 C CNN
 F 1 "4.7k" V 8700 3750 50  0000 C CNN
-F 2 "Resistor_SMD:R_0603_1608Metric" H 8700 3750 60  0001 C CNN
+F 2 "Resistor_SMD:R_0402_1005Metric" H 8700 3750 60  0001 C CNN
 F 3 "" H 8700 3750 60  0001 C CNN
 	1    8700 3750
@@
 F 0 "R51" V 6050 4700 50  0000 C CNN
 F 1 "4.7k" V 6150 4700 50  0000 C CNN
-F 2 "Resistor_SMD:R_0603_1608Metric" H 6150 4700 60  0001 C CNN
+F 2 "Resistor_SMD:R_0402_1005Metric" H 6150 4700 60  0001 C CNN
 F 3 "" H 6150 4700 60  0001 C CNN
 	1    6150 4700
@@
 F 0 "R37" V 7300 4800 50  0000 C CNN
 F 1 "10R" V 7100 4800 50  0000 C CNN
-F 2 "Resistor_SMD:R_0805_2012Metric" H 7200 4800 60  0001 C CNN
+F 2 "Resistor_SMD:R_0402_1005Metric" H 7200 4800 60  0001 C CNN
 F 3 "" H 7200 4800 60  0001 C CNN
 	1    7200 4800
@@
 F 0 "C61" H 3400 3450 50  0000 L CNN
 F 1 "1nF" H 3400 3250 50  0000 L CNN
-F 2 "Capacitor_SMD:C_0603_1608Metric" H 3400 3350 60  0001 C CNN
+F 2 "Capacitor_SMD:C_0402_1005Metric" H 3400 3350 60  0001 C CNN
 F 3 "" H 3400 3350 60  0001 C CNN
 	1    3400 3350
@@
 F 0 "C62" H 3400 4400 50  0000 L CNN
 F 1 "1nF" H 3400 4200 50  0000 L CNN
-F 2 "Capacitor_SMD:C_0603_1608Metric" H 3400 4300 60  0001 C CNN
+F 2 "Capacitor_SMD:C_0402_1005Metric" H 3400 4300 60  0001 C CNN
 F 3 "" H 3400 4300 60  0001 C CNN
 	1    3400 4300
@@
 F 0 "C65" H 6050 4450 50  0000 L CNN
 F 1 "1nF" H 6050 4250 50  0000 L CNN
-F 2 "Capacitor_SMD:C_0603_1608Metric" H 6050 4350 60  0001 C CNN
+F 2 "Capacitor_SMD:C_0402_1005Metric" H 6050 4350 60  0001 C CNN
 F 3 "" H 6050 4350 60  0001 C CNN
 	1    6050 4350
@@
 F 0 "C63" H 6050 3500 50  0000 L CNN
 F 1 "1nF" H 6050 3300 50  0000 L CNN
-F 2 "Capacitor_SMD:C_0603_1608Metric" H 6050 3400 60  0001 C CNN
+F 2 "Capacitor_SMD:C_0402_1005Metric" H 6050 3400 60  0001 C CNN
 F 3 "" H 6050 3400 60  0001 C CNN
 	1    6050 3400
@@
 F 0 "C66" H 8600 3550 50  0000 L CNN
 F 1 "1nF" H 8600 3350 50  0000 L CNN
-F 2 "Capacitor_SMD:C_0603_1608Metric" H 8600 3450 60  0001 C CNN
+F 2 "Capacitor_SMD:C_0402_1005Metric" H 8600 3450 60  0001 C CNN
 F 3 "" H 8600 3450 60  0001 C CNN
 	1    8600 3450
@@
 F 0 "C67" H 8600 4500 50  0000 L CNN
 F 1 "1nF" H 8600 4300 50  0000 L CNN
-F 2 "Capacitor_SMD:C_0603_1608Metric" H 8600 4400 60  0001 C CNN
+F 2 "Capacitor_SMD:C_0402_1005Metric" H 8600 4400 60  0001 C CNN
 F 3 "" H 8600 4400 60  0001 C CNN
 	1    8600 4400
@@
 F 0 "R45" V 6050 3750 50  0000 C CNN
 F 1 "4.7k" V 6150 3750 50  0000 C CNN
-F 2 "Resistor_SMD:R_0603_1608Metric" H 6150 3750 60  0001 C CNN
+F 2 "Resistor_SMD:R_0402_1005Metric" H 6150 3750 60  0001 C CNN
 F 3 "" H 6150 3750 60  0001 C CNN
 	1    6150 3750
