File: source/temp.sch (KiCad schematic (older format))
At the start: 3 parts

Commit message: started redrawing pcb
Parts:
- C5: footprint Capacitor_SMD:C_0603_1608Metric -> Capacitor_SMD:C_0402_1005Metric
- R13: footprint Resistor_SMD:R_0603_1608Metric -> Resistor_SMD:R_0402_1005Metric
Changed lines of the file:
@@
 $Descr A4 11693 8268
 encoding utf-8
-Sheet 2 8
+Sheet 2 6
 Title "Cheap FOCer 2"
 Date "2020-04-08"
@@
 F 0 "R13" V 5880 4000 40  0000 C CNN
 F 1 "10k" V 5807 4001 40  0000 C CNN
-F 2 "Resistor_SMD:R_0603_1608Metric" V 5730 4000 30  0001 C CNN
+F 2 "Resistor_SMD:R_0402_1005Metric" V 5730 4000 30  0001 C CNN
 F 3 "" H 5800 4000 30  0000 C CNN
 	1    5800 4000
@@
 F 0 "C5" H 5550 4100 40  0000 L CNN
 F 1 "2.2u" H 5556 3915 40  0000 L CNN
-F 2 "Capacitor_SMD:C_0603_1608Metric" H 5588 3850 30  0001 C CNN
+F 2 "Capacitor_SMD:C_0402_1005Metric" H 5588 3850 30  0001 C CNN
 F 3 "" H 5550 4000 60  0000 C CNN
 	1    5550 4000
