File: source/IMU.sch (KiCad schematic (older format))
At the start: 5 parts, among them U6 BMI160

Commit message: Put back Q6 which was accidentally deleted
Parts:
- U6: symbol Cheap-FOCer-2-60mm-rescue:BMI160-IMU -> Cheap-FOCer-2-60mm-rescue:BMI160-IMU-Cheap-FOCer-2-60mm-rescue
Changed lines of the file:
@@
 $EndComp
 $Comp
-L Cheap-FOCer-2-60mm-rescue:BMI160-IMU U6
+L Cheap-FOCer-2-60mm-rescue:BMI160-IMU-Cheap-FOCer-2-60mm-rescue U6
 U 1 1 5E6217EF
 P 4300 3300
