File: source/IMU.sch (KiCad schematic (older format))
At the start: 5 parts, among them U6 BMI160

Commit message: Revert "Remove transistors"
Parts:
- U6: symbol Cheap-FOCer-2-60mm-rescue:BMI160-IMU-Cheap-FOCer-2-60mm-rescue -> Cheap-FOCer-2-60mm-rescue:BMI160-IMU
Changed lines of the file:
@@
 Sheet 7 8
 Title "Cheap FOCer 2"
-Date "2021-06-25"
-Rev "1.0"
+Date "2020-04-08"
+Rev "0.9"
 Comp "Shaman Systems"
 Comment1 "Root"
@@
 $EndComp
 $Comp
-L Cheap-FOCer-2-60mm-rescue:BMI160-IMU-Cheap-FOCer-2-60mm-rescue U6
+L Cheap-FOCer-2-60mm-rescue:BMI160-IMU U6
 U 1 1 5E6217EF
 P 4300 3300

Commit message: Removed gate transistors
Parts:
- U6: symbol Cheap-FOCer-2-60mm-rescue:BMI160-IMU -> Cheap-FOCer-2-60mm-rescue:BMI160-IMU-Cheap-FOCer-2-60mm-rescue
Changed lines of the file:
@@
 Sheet 7 8
 Title "Cheap FOCer 2"
-Date "2020-04-08"
-Rev "0.9"
+Date "2021-06-25"
+Rev "1.0"
 Comp "Shaman Systems"
 Comment1 "Root"
@@
 $EndComp
 $Comp
-L Cheap-FOCer-2-60mm-rescue:BMI160-IMU U6
+L Cheap-FOCer-2-60mm-rescue:BMI160-IMU-Cheap-FOCer-2-60mm-rescue U6
 U 1 1 5E6217EF
 P 4300 3300
